File: 20210227 - B+ to VM/B+ to VM Protection Circuit.sch (EAGLE design)
At the start: 46 parts, among them Q1 SOT23, Q4 SOT23, Q5 DPACK

Commit message: 02MAR2021
Parts:
- added NM.02MAR2021: VM FILTER, NMOS-SOURCE-FOLLOWER, nolan:PCB_EVAL_80X80
- added TP10, TP11, TP12, TP13, TP14, TP8, TP9: TESTPOINTKE5000-SMTEXT, nolan:TESTPOINTKE5000-SMTEXT
- added U$1, U$2: SPADE-TAB, nolan:SPADE-TAB
- C2: value 0805 -> PCR-10X8; device nolan:C-EUC0805 -> nolan:C-EUPCR-10X8
- C4: value PCR-10X8 -> 1206; device nolan:C-EUPCR-10X8 -> nolan:C-EUC1206
- C5: value 1206 -> 0805; device nolan:C-EUC1206 -> nolan:C-EUC0805
- C7: value PCR-8X7 -> 1206; device nolan:C-EUPCR-8X7 -> nolan:C-EUC1206
- C8: value PCR-10X8 -> PCR-8X7; device nolan:C-EUPCR-10X8 -> nolan:C-EUPCR-8X7
- C9: value 1206 -> PCR-10X8; device nolan:C-EUC1206 -> nolan:C-EUPCR-10X8
- R19: device nolan:R-EU_M2012 -> nolan:R-EU_R1210
- R5, R6, R8, R9: device nolan:R-EU_0207/10 -> nolan:R-EU_M0805
- TP1, TP2, TP3, TP4, TP5, TP6, TP7: value TESTPOINTKE5000 -> TESTPOINTKE5000-SMTEXT; device nolan:TESTPOINTKE5000 -> nolan:TESTPOINTKE5000-SMTEXT
Connections:
- net B+: now also TP7.1; no longer TP4.1
- net GND: now also NM.02MAR2021.GND, R11.2, R18.2, R5.1, TP4.1, TP5.1, TP6.1; no longer R14.2, R17.2, R7.1
- net HIGH_VOLTAGE: now also NM.02MAR2021.V1+, R13.1; no longer R12.1
- net HIGH_VOLTAGE_CONTROL_1: now also R11.1, R12.1, TP13.1; no longer R13.1, R14.1
- net LOAD_CONTROL_1: now also R5.2, R6.2, TP9.1; no longer R10.2, R7.2
- net LOAD_CONTROL_2: now also TP11.1
- net N$10: now also D3.A, R18.1; no longer D4.A, R15.1
- net N$11: now also R17.2; no longer R16.2
- net N$12: now also D4.A, U$2.P$1; no longer D3.A
- net N$13: now also R16.1; no longer R11.1
- net N$2: now also R7.1, TP10.1; no longer R5.1, TP5.1
- net N$3: now also R10.1, TP12.1; no longer R6.1, TP6.1
- net N$6: now also R6.1; no longer R10.1
- net N$7: now also R13.2, R14.1, R16.2; no longer R11.2, R12.2, R18.1
- net N$8: now also R12.2; no longer R13.2
- net N$9: now also R14.2; no longer R18.2
- net SPIKE_VOLTAGE_CONTROL_2: now also R15.1, TP14.1; no longer R16.1
- net VIN: now also NM.02MAR2021.V2+, U$1.P$1
- net VM: now also R10.2, R7.2, TP8.1; no longer R5.2, R6.2, TP7.1
Other:
- moved on the sheet: C2, C4, C5, C7, C8, C9, D3, D4, L1, Q6, R10, R11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

Commit message: 02MAR2021
Parts:
- NM.02MAR2021: value VM FILTER, NMOS-SOURCE-FOLLOWER -> B+ TO VM FILTER, NMOS-SOURCE-FOLLOWER
Changed lines of the file:
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@@
 <part name="U$1" library="nolan" deviceset="SPADE-TAB" device=""/>
 <part name="U$2" library="nolan" deviceset="SPADE-TAB" device=""/>
-<part name="NM.02MAR2021" library="nolan" deviceset="PCB_EVAL_80X80" device="" value="VM FILTER, NMOS-SOURCE-FOLLOWER"/>
+<part name="NM.02MAR2021" library="nolan" deviceset="PCB_EVAL_80X80" device="" value="B+ TO VM FILTER, NMOS-SOURCE-FOLLOWER"/>
 <part name="TP9" library="nolan" deviceset="TESTPOINT" device="KE5000-SMTEXT"/>
 <part name="TP11" library="nolan" deviceset="TESTPOINT" device="KE5000-SMTEXT"/>
