File: 202103 - Capacitor Thermal Gradient/Capacitor Thermal Gradient Test Board.brd (EAGLE design)
At the start: 11 parts, among them Q1 RYC002N05T316

Commit message: 20210303
Parts:
- removed 1.GND, 2.PWR, 3.OUT: TESTPOINTKE5000-SMTEXT, nolan:PINS_1_TESTPOINT_KE5000_NOTEXT
- removed C5, C6: 4u7 50V, nolan:C0805
- removed D2: SM4001PL, nolan:SOD123
- removed Q1: RYC002N05T316, nolan:SOT23
- removed ZD1: 15V, nolan:SOT23
- added C2: C-EU_10X5, nolan:C_PZF_10
- added P1, P2, P3, P4: (no value), nolan:PINS_1_2MM2
- C1: value 1u -> C-EU_10X5; device nolan:C0402 -> nolan:C_PZF_10
- R1: value 10k -> (none); device nolan:R0402 -> nolan:R_THERMAL_1225
- R2: value 499k -> (none); device nolan:R0402 -> nolan:R_THERMAL_1225
- moved C1 38.0 mm to (36.0, 25.0), turned to 90 degrees
- moved R1 29.6 mm to (31.0, 25.0), flipped to the bottom, turned to 90 degrees
- moved R2 24.2 mm to (19.0, 25.0), flipped to the bottom, turned to 90 degrees
Connections:
- removed net B+: 2.PWR.1, D2.A
- removed net GND: 1.GND.1, C1.2, C5.2, C6.2, R2.1, ZD1.1
- removed net Q1.DRAIN: C5.1, C6.1, D2.C, Q1.3, R1.2
- removed net Q1.GATE: C1.1, Q1.1, R1.1, R2.2, ZD1.3
- removed net VM: 3.OUT.1, Q1.2
- new net N$1: C1.1+, P1.1, R1.2
- new net N$2: C1.2-, P2.1, R1.1
- new net N$3: C2.1+, P3.1, R2.2
- new net N$4: C2.2-, P4.1, R2.1
Routing:
- net N$4: track 0.00 -> 18.5 mm, vias 0 -> 5
- net N$3: track 0.00 -> 18.5 mm, vias 0 -> 5
- net N$2: track 0.00 -> 18.5 mm, vias 0 -> 5
- net N$1: track 0.00 -> 18.5 mm, vias 0 -> 5
- net GND: track 17.6 -> 0.00 mm
- net Q1.DRAIN: track 9.10 -> 0.00 mm, vias 1 -> 0
- net Q1.GATE: track 7.21 -> 0.00 mm
- net VM: track 3.50 -> 0.00 mm
- net B+: track 2.09 -> 0.00 mm
- added copper zone on layer 1, net N$1
- added copper zone on layer 16, net N$1
- added copper zone on layer 1, net N$2
- added copper zone on layer 16, net N$2
- added copper zone on layer 1, net N$3
- added copper zone on layer 16, net N$3
- added copper zone on layer 1, net N$4
- added copper zone on layer 16, net N$4
Other:
- board text added: "C2"
- board text added: "CAPACITORS: 10mm diameter, 5mm pitch"
- board text added: "NM.03MAR2021"
- board text added: "P1"
- board text added: "P2"
- board text added: "P3"
- board text added: "P4"
- board text added: "THERMAL GRADIENT EXPERIMENT BOARD"
- board text added: "THERMAWICK: THJP1225AST1"
- board text removed: "1.GND"
- board text removed: "3.OUT"
- board text removed: "C5"
- board text removed: "C6"
- board text removed: "D2"
- board text removed: "Q1"
- board text removed: "ZD1"
