File: 202103 - DIY Dyno/DIY Dyno.sch (EAGLE design)
At the start: 0 parts

Commit message: 20210310
Other:
- note added: "LOAD -- 2400W 170mOhm"
- note removed: "LOAD -- 3200W 130mOhm"
Changed lines of the file:
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@@
 <text x="231.14" y="142.24" size="2.54" layer="94" align="center">LOAD
 --
-3200W
-130mOhm</text>
+2400W
+170mOhm</text>
 <text x="147.32" y="137.16" size="2.54" layer="94" align="center">U</text>
 <text x="147.32" y="132.08" size="2.54" layer="94" align="center">V</text>
