File: VM Protection Circuit/panel.brd (EAGLE design)
At the start: 100 x 90 mm, 660 parts, among them Q1 RYC002N05T316, Q10 RYC002N05T316, Q11 RYC002N05T316, Q12 RYC002N05T316, Q13 RYC002N05T316, Q14 RYC002N05T316, Q15 RYC002N05T316, Q16 RYC002N05T316, Q17 RYC002N05T316, Q18 RYC002N05T316, Q19 RYC002N05T316, Q2 RYC002N05T316, Q20 RYC002N05T316, Q21 RYC002N05T316, Q22 RYC002N05T316, Q23 RYC002N05T316, Q24 RYC002N05T316, Q25 RYC002N05T316, Q26 RYC002N05T316, Q27 RYC002N05T316, Q28 RYC002N05T316, Q29 RYC002N05T316, Q3 RYC002N05T316, Q30 RYC002N05T316, Q31 RYC002N05T316, Q32 RYC002N05T316, Q33 RYC002N05T316, Q34 RYC002N05T316, Q35 RYC002N05T316, Q36 RYC002N05T316, Q37 RYC002N05T316, Q38 RYC002N05T316, Q39 RYC002N05T316, Q4 RYC002N05T316, Q40 RYC002N05T316, Q41 RYC002N05T316, Q42 RYC002N05T316, Q5 RYC002N05T316, Q55 RYC002N05T316, Q56 RYC002N05T316, Q57 RYC002N05T316, Q58 RYC002N05T316, Q59 RYC002N05T316, Q6 RYC002N05T316, Q60 RYC002N05T316, Q61 RYC002N05T316, Q62 RYC002N05T316, Q63 RYC002N05T316, Q64 RYC002N05T316, Q65 RYC002N05T316, Q66 RYC002N05T316, Q67 RYC002N05T316, Q68 RYC002N05T316, Q69 RYC002N05T316, Q7 RYC002N05T316, Q70 RYC002N05T316, Q71 RYC002N05T316, Q72 RYC002N05T316, Q8 RYC002N05T316, Q9 RYC002N05T316

Commit message: 20210313
Parts:
- removed 1.GND10, 1.GND11, 1.GND16, 1.GND17, 1.GND22, 1.GND23, 1.GND24, 1.GND25, 1.GND26, 1.GND27, 1.GND28, 1.GND29, 1.GND30, 1.GND31, 1.GND32, 1.GND33, 1.GND34, 1.GND35, 1.GND36, 1.GND37, 1.GND38, 1.GND39, 1.GND4, 1.GND40, 1.GND41, 1.GND5, 1.GND54, 1.GND55, 1.GND56, 1.GND57, 1.GND58, 1.GND59, 1.GND60, 1.GND61, 1.GND62, 1.GND63, 1.GND64, 1.GND65, 1.GND66, 1.GND67, 1.GND68, 1.GND69, 1.GND70, 1.GND71, 2.PWR10, 2.PWR11, 2.PWR16, 2.PWR17, 2.PWR22, 2.PWR23, 2.PWR24, 2.PWR25, 2.PWR26, 2.PWR27, 2.PWR28, 2.PWR29, 2.PWR30, 2.PWR31, 2.PWR32, 2.PWR33, 2.PWR34, 2.PWR35, 2.PWR36, 2.PWR37, 2.PWR38, 2.PWR39, 2.PWR4, 2.PWR40, 2.PWR41, 2.PWR5, 2.PWR54, 2.PWR55, 2.PWR56, 2.PWR57, 2.PWR58, 2.PWR59, 2.PWR60, 2.PWR61, 2.PWR62, 2.PWR63, 2.PWR64, 2.PWR65, 2.PWR66, 2.PWR67, 2.PWR68, 2.PWR69, 2.PWR70, 2.PWR71, 3.OUT10, 3.OUT11, 3.OUT16, 3.OUT17, 3.OUT22, 3.OUT23, 3.OUT24, 3.OUT25, 3.OUT26, 3.OUT27, 3.OUT28, 3.OUT29, 3.OUT30, 3.OUT31, 3.OUT32, 3.OUT33, 3.OUT34, 3.OUT35, 3.OUT36, 3.OUT37, 3.OUT38, 3.OUT39, 3.OUT4, 3.OUT40, 3.OUT41, 3.OUT5, 3.OUT54, 3.OUT55, 3.OUT56, 3.OUT57, 3.OUT58, 3.OUT59, 3.OUT60, 3.OUT61, 3.OUT62, 3.OUT63, 3.OUT64, 3.OUT65, 3.OUT66, 3.OUT67, 3.OUT68, 3.OUT69, 3.OUT70, 3.OUT71: TESTPOINTKE5000-SMTEXT, nolan:PINS_1_TESTPOINT_KE5000_NOTEXT
- removed C100, C103, C106, C109, C112, C115, C118, C121, C124, C13, C16, C163, C166, C169, C172, C175, C178, C181, C184, C187, C190, C193, C196, C199, C202, C205, C208, C211, C214, C31, C34, C49, C52, C67, C70, C73, C76, C79, C82, C85, C88, C91, C94, C97: 1u, nolan:C0402
- removed C101, C102, C104, C105, C107, C108, C110, C111, C113, C114, C116, C117, C119, C120, C122, C123, C125, C126, C14, C15, C164, C165, C167, C168, C17, C170, C171, C173, C174, C176, C177, C179, C18, C180, C182, C183, C185, C186, C188, C189, C191, C192, C194, C195, C197, C198, C200, C201, C203, C204, C206, C207, C209, C210, C212, C213, C215, C216, C32, C33, C35, C36, C50, C51, C53, C54, C68, C69, C71, C72, C74, C75, C77, C78, C80, C81, C83, C84, C86, C87, C89, C90, C92, C93, C95, C96, C98, C99: 4u7 50V, nolan:C0805
- removed D11, D12, D17, D18, D23, D24, D25, D26, D27, D28, D29, D30, D31, D32, D33, D34, D35, D36, D37, D38, D39, D40, D41, D42, D5, D55, D56, D57, D58, D59, D6, D60, D61, D62, D63, D64, D65, D66, D67, D68, D69, D70, D71, D72: SM4001PL, nolan:SOD123
- removed Q11, Q12, Q17, Q18, Q23, Q24, Q25, Q26, Q27, Q28, Q29, Q30, Q31, Q32, Q33, Q34, Q35, Q36, Q37, Q38, Q39, Q40, Q41, Q42, Q5, Q55, Q56, Q57, Q58, Q59, Q6, Q60, Q61, Q62, Q63, Q64, Q65, Q66, Q67, Q68, Q69, Q70, Q71, Q72: RYC002N05T316, nolan:SOT23
- removed R10, R110, R112, R114, R116, R118, R12, R120, R122, R124, R126, R128, R130, R132, R134, R136, R138, R140, R142, R144, R22, R24, R34, R36, R46, R48, R50, R52, R54, R56, R58, R60, R62, R64, R66, R68, R70, R72, R74, R76, R78, R80, R82, R84: 499k, nolan:R0402
- removed R109, R11, R111, R113, R115, R117, R119, R121, R123, R125, R127, R129, R131, R133, R135, R137, R139, R141, R143, R21, R23, R33, R35, R45, R47, R49, R51, R53, R55, R57, R59, R61, R63, R65, R67, R69, R71, R73, R75, R77, R79, R81, R83, R9: 10k, nolan:R0402
- removed ZD11, ZD12, ZD17, ZD18, ZD23, ZD24, ZD25, ZD26, ZD27, ZD28, ZD29, ZD30, ZD31, ZD32, ZD33, ZD34, ZD35, ZD36, ZD37, ZD38, ZD39, ZD40, ZD41, ZD42, ZD5, ZD55, ZD56, ZD57, ZD58, ZD59, ZD6, ZD60, ZD61, ZD62, ZD63, ZD64, ZD65, ZD66, ZD67, ZD68, ZD69, ZD70, ZD71, ZD72: 15V, nolan:SOT23
Connections:
- removed net B+10: 2.PWR10.1, D11.A
- removed net B+11: 2.PWR11.1, D12.A
- removed net B+16: 2.PWR16.1, D17.A
- removed net B+17: 2.PWR17.1, D18.A
- removed net B+22: 2.PWR22.1, D23.A
- removed net B+23: 2.PWR23.1, D24.A
- removed net B+24: 2.PWR24.1, D25.A
- removed net B+25: 2.PWR25.1, D26.A
- removed net B+26: 2.PWR26.1, D27.A
- removed net B+27: 2.PWR27.1, D28.A
- removed net B+28: 2.PWR28.1, D29.A
- removed net B+29: 2.PWR29.1, D30.A
- removed net B+30: 2.PWR30.1, D31.A
- removed net B+31: 2.PWR31.1, D32.A
- removed net B+32: 2.PWR32.1, D33.A
- removed net B+33: 2.PWR33.1, D34.A
- removed net B+34: 2.PWR34.1, D35.A
- removed net B+35: 2.PWR35.1, D36.A
- removed net B+36: 2.PWR36.1, D37.A
- removed net B+37: 2.PWR37.1, D38.A
- removed net B+38: 2.PWR38.1, D39.A
- removed net B+39: 2.PWR39.1, D40.A
- removed net B+4: 2.PWR4.1, D5.A
- removed net B+40: 2.PWR40.1, D41.A
- removed net B+41: 2.PWR41.1, D42.A
- removed net B+5: 2.PWR5.1, D6.A
- removed net B+54: 2.PWR54.1, D55.A
- removed net B+55: 2.PWR55.1, D56.A
- removed net B+56: 2.PWR56.1, D57.A
- removed net B+57: 2.PWR57.1, D58.A
- removed net B+58: 2.PWR58.1, D59.A
- removed net B+59: 2.PWR59.1, D60.A
- removed net B+60: 2.PWR60.1, D61.A
- removed net B+61: 2.PWR61.1, D62.A
- removed net B+62: 2.PWR62.1, D63.A
- removed net B+63: 2.PWR63.1, D64.A
- removed net B+64: 2.PWR64.1, D65.A
- removed net B+65: 2.PWR65.1, D66.A
- removed net B+66: 2.PWR66.1, D67.A
- removed net B+67: 2.PWR67.1, D68.A
- removed net B+68: 2.PWR68.1, D69.A
- removed net B+69: 2.PWR69.1, D70.A
- removed net B+70: 2.PWR70.1, D71.A
- removed net B+71: 2.PWR71.1, D72.A
- removed net GND10: 1.GND10.1, C31.2, C32.2, C33.2, R22.1, ZD11.1
- removed net GND11: 1.GND11.1, C34.2, C35.2, C36.2, R24.1, ZD12.1
- removed net GND16: 1.GND16.1, C49.2, C50.2, C51.2, R34.1, ZD17.1
- removed net GND17: 1.GND17.1, C52.2, C53.2, C54.2, R36.1, ZD18.1
- removed net GND22: 1.GND22.1, C67.2, C68.2, C69.2, R46.1, ZD23.1
- removed net GND23: 1.GND23.1, C70.2, C71.2, C72.2, R48.1, ZD24.1
- removed net GND24: 1.GND24.1, C73.2, C74.2, C75.2, R50.1, ZD25.1
- removed net GND25: 1.GND25.1, C76.2, C77.2, C78.2, R52.1, ZD26.1
- removed net GND26: 1.GND26.1, C79.2, C80.2, C81.2, R54.1, ZD27.1
- removed net GND27: 1.GND27.1, C82.2, C83.2, C84.2, R56.1, ZD28.1
- removed net GND28: 1.GND28.1, C85.2, C86.2, C87.2, R58.1, ZD29.1
- removed net GND29: 1.GND29.1, C88.2, C89.2, C90.2, R60.1, ZD30.1
- removed net GND30: 1.GND30.1, C91.2, C92.2, C93.2, R62.1, ZD31.1
- removed net GND31: 1.GND31.1, C94.2, C95.2, C96.2, R64.1, ZD32.1
- removed net GND32: 1.GND32.1, C97.2, C98.2, C99.2, R66.1, ZD33.1
- removed net GND33: 1.GND33.1, C100.2, C101.2, C102.2, R68.1, ZD34.1
- removed net GND34: 1.GND34.1, C103.2, C104.2, C105.2, R70.1, ZD35.1
- removed net GND35: 1.GND35.1, C106.2, C107.2, C108.2, R72.1, ZD36.1
- removed net GND36: 1.GND36.1, C109.2, C110.2, C111.2, R74.1, ZD37.1
- removed net GND37: 1.GND37.1, C112.2, C113.2, C114.2, R76.1, ZD38.1
- removed net GND38: 1.GND38.1, C115.2, C116.2, C117.2, R78.1, ZD39.1
- removed net GND39: 1.GND39.1, C118.2, C119.2, C120.2, R80.1, ZD40.1
- removed net GND4: 1.GND4.1, C13.2, C14.2, C15.2, R10.1, ZD5.1
- removed net GND40: 1.GND40.1, C121.2, C122.2, C123.2, R82.1, ZD41.1
- removed net GND41: 1.GND41.1, C124.2, C125.2, C126.2, R84.1, ZD42.1
- removed net GND5: 1.GND5.1, C16.2, C17.2, C18.2, R12.1, ZD6.1
- removed net GND54: 1.GND54.1, C163.2, C164.2, C165.2, R110.1, ZD55.1
- removed net GND55: 1.GND55.1, C166.2, C167.2, C168.2, R112.1, ZD56.1
- removed net GND56: 1.GND56.1, C169.2, C170.2, C171.2, R114.1, ZD57.1
- removed net GND57: 1.GND57.1, C172.2, C173.2, C174.2, R116.1, ZD58.1
- removed net GND58: 1.GND58.1, C175.2, C176.2, C177.2, R118.1, ZD59.1
- removed net GND59: 1.GND59.1, C178.2, C179.2, C180.2, R120.1, ZD60.1
- removed net GND60: 1.GND60.1, C181.2, C182.2, C183.2, R122.1, ZD61.1
- removed net GND61: 1.GND61.1, C184.2, C185.2, C186.2, R124.1, ZD62.1
- removed net GND62: 1.GND62.1, C187.2, C188.2, C189.2, R126.1, ZD63.1
- removed net GND63: 1.GND63.1, C190.2, C191.2, C192.2, R128.1, ZD64.1
- removed net GND64: 1.GND64.1, C193.2, C194.2, C195.2, R130.1, ZD65.1
- removed net GND65: 1.GND65.1, C196.2, C197.2, C198.2, R132.1, ZD66.1
- removed net GND66: 1.GND66.1, C199.2, C200.2, C201.2, R134.1, ZD67.1
- removed net GND67: 1.GND67.1, C202.2, C203.2, C204.2, R136.1, ZD68.1
- removed net GND68: 1.GND68.1, C205.2, C206.2, C207.2, R138.1, ZD69.1
- removed net GND69: 1.GND69.1, C208.2, C209.2, C210.2, R140.1, ZD70.1
- removed net GND70: 1.GND70.1, C211.2, C212.2, C213.2, R142.1, ZD71.1
- removed net GND71: 1.GND71.1, C214.2, C215.2, C216.2, R144.1, ZD72.1
- removed net Q1.DRAIN10: C32.1, C33.1, D11.C, Q11.3, R21.2
- removed net Q1.DRAIN11: C35.1, C36.1, D12.C, Q12.3, R23.2
- removed net Q1.DRAIN16: C50.1, C51.1, D17.C, Q17.3, R33.2
- removed net Q1.DRAIN17: C53.1, C54.1, D18.C, Q18.3, R35.2
- removed net Q1.DRAIN22: C68.1, C69.1, D23.C, Q23.3, R45.2
- removed net Q1.DRAIN23: C71.1, C72.1, D24.C, Q24.3, R47.2
- removed net Q1.DRAIN24: C74.1, C75.1, D25.C, Q25.3, R49.2
- removed net Q1.DRAIN25: C77.1, C78.1, D26.C, Q26.3, R51.2
- removed net Q1.DRAIN26: C80.1, C81.1, D27.C, Q27.3, R53.2
- removed net Q1.DRAIN27: C83.1, C84.1, D28.C, Q28.3, R55.2
- removed net Q1.DRAIN28: C86.1, C87.1, D29.C, Q29.3, R57.2
- removed net Q1.DRAIN29: C89.1, C90.1, D30.C, Q30.3, R59.2
- removed net Q1.DRAIN30: C92.1, C93.1, D31.C, Q31.3, R61.2
- removed net Q1.DRAIN31: C95.1, C96.1, D32.C, Q32.3, R63.2
- removed net Q1.DRAIN32: C98.1, C99.1, D33.C, Q33.3, R65.2
- removed net Q1.DRAIN33: C101.1, C102.1, D34.C, Q34.3, R67.2
- removed net Q1.DRAIN34: C104.1, C105.1, D35.C, Q35.3, R69.2
- removed net Q1.DRAIN35: C107.1, C108.1, D36.C, Q36.3, R71.2
- removed net Q1.DRAIN36: C110.1, C111.1, D37.C, Q37.3, R73.2
- removed net Q1.DRAIN37: C113.1, C114.1, D38.C, Q38.3, R75.2
- removed net Q1.DRAIN38: C116.1, C117.1, D39.C, Q39.3, R77.2
- removed net Q1.DRAIN39: C119.1, C120.1, D40.C, Q40.3, R79.2
- removed net Q1.DRAIN4: C14.1, C15.1, D5.C, Q5.3, R9.2
- removed net Q1.DRAIN40: C122.1, C123.1, D41.C, Q41.3, R81.2
- removed net Q1.DRAIN41: C125.1, C126.1, D42.C, Q42.3, R83.2
- removed net Q1.DRAIN5: C17.1, C18.1, D6.C, Q6.3, R11.2
- removed net Q1.DRAIN54: C164.1, C165.1, D55.C, Q55.3, R109.2
- removed net Q1.DRAIN55: C167.1, C168.1, D56.C, Q56.3, R111.2
- removed net Q1.DRAIN56: C170.1, C171.1, D57.C, Q57.3, R113.2
- removed net Q1.DRAIN57: C173.1, C174.1, D58.C, Q58.3, R115.2
- removed net Q1.DRAIN58: C176.1, C177.1, D59.C, Q59.3, R117.2
- removed net Q1.DRAIN59: C179.1, C180.1, D60.C, Q60.3, R119.2
- removed net Q1.DRAIN60: C182.1, C183.1, D61.C, Q61.3, R121.2
- removed net Q1.DRAIN61: C185.1, C186.1, D62.C, Q62.3, R123.2
- removed net Q1.DRAIN62: C188.1, C189.1, D63.C, Q63.3, R125.2
- removed net Q1.DRAIN63: C191.1, C192.1, D64.C, Q64.3, R127.2
- removed net Q1.DRAIN64: C194.1, C195.1, D65.C, Q65.3, R129.2
- removed net Q1.DRAIN65: C197.1, C198.1, D66.C, Q66.3, R131.2
- removed net Q1.DRAIN66: C200.1, C201.1, D67.C, Q67.3, R133.2
- removed net Q1.DRAIN67: C203.1, C204.1, D68.C, Q68.3, R135.2
- removed net Q1.DRAIN68: C206.1, C207.1, D69.C, Q69.3, R137.2
- removed net Q1.DRAIN69: C209.1, C210.1, D70.C, Q70.3, R139.2
- removed net Q1.DRAIN70: C212.1, C213.1, D71.C, Q71.3, R141.2
- removed net Q1.DRAIN71: C215.1, C216.1, D72.C, Q72.3, R143.2
- removed net Q1.GATE10: C31.1, Q11.1, R21.1, R22.2, ZD11.3
- removed net Q1.GATE11: C34.1, Q12.1, R23.1, R24.2, ZD12.3
- removed net Q1.GATE16: C49.1, Q17.1, R33.1, R34.2, ZD17.3
- removed net Q1.GATE17: C52.1, Q18.1, R35.1, R36.2, ZD18.3
- removed net Q1.GATE22: C67.1, Q23.1, R45.1, R46.2, ZD23.3
- removed net Q1.GATE23: C70.1, Q24.1, R47.1, R48.2, ZD24.3
- removed net Q1.GATE24: C73.1, Q25.1, R49.1, R50.2, ZD25.3
- removed net Q1.GATE25: C76.1, Q26.1, R51.1, R52.2, ZD26.3
- removed net Q1.GATE26: C79.1, Q27.1, R53.1, R54.2, ZD27.3
- removed net Q1.GATE27: C82.1, Q28.1, R55.1, R56.2, ZD28.3
- removed net Q1.GATE28: C85.1, Q29.1, R57.1, R58.2, ZD29.3
- removed net Q1.GATE29: C88.1, Q30.1, R59.1, R60.2, ZD30.3
- removed net Q1.GATE30: C91.1, Q31.1, R61.1, R62.2, ZD31.3
- removed net Q1.GATE31: C94.1, Q32.1, R63.1, R64.2, ZD32.3
- removed net Q1.GATE32: C97.1, Q33.1, R65.1, R66.2, ZD33.3
- removed net Q1.GATE33: C100.1, Q34.1, R67.1, R68.2, ZD34.3
- removed net Q1.GATE34: C103.1, Q35.1, R69.1, R70.2, ZD35.3
- removed net Q1.GATE35: C106.1, Q36.1, R71.1, R72.2, ZD36.3
- removed net Q1.GATE36: C109.1, Q37.1, R73.1, R74.2, ZD37.3
- removed net Q1.GATE37: C112.1, Q38.1, R75.1, R76.2, ZD38.3
- removed net Q1.GATE38: C115.1, Q39.1, R77.1, R78.2, ZD39.3
- removed net Q1.GATE39: C118.1, Q40.1, R79.1, R80.2, ZD40.3
- removed net Q1.GATE4: C13.1, Q5.1, R10.2, R9.1, ZD5.3
- removed net Q1.GATE40: C121.1, Q41.1, R81.1, R82.2, ZD41.3
- removed net Q1.GATE41: C124.1, Q42.1, R83.1, R84.2, ZD42.3
- removed net Q1.GATE5: C16.1, Q6.1, R11.1, R12.2, ZD6.3
- removed net Q1.GATE54: C163.1, Q55.1, R109.1, R110.2, ZD55.3
- removed net Q1.GATE55: C166.1, Q56.1, R111.1, R112.2, ZD56.3
- removed net Q1.GATE56: C169.1, Q57.1, R113.1, R114.2, ZD57.3
- removed net Q1.GATE57: C172.1, Q58.1, R115.1, R116.2, ZD58.3
- removed net Q1.GATE58: C175.1, Q59.1, R117.1, R118.2, ZD59.3
- removed net Q1.GATE59: C178.1, Q60.1, R119.1, R120.2, ZD60.3
- removed net Q1.GATE60: C181.1, Q61.1, R121.1, R122.2, ZD61.3
- removed net Q1.GATE61: C184.1, Q62.1, R123.1, R124.2, ZD62.3
- removed net Q1.GATE62: C187.1, Q63.1, R125.1, R126.2, ZD63.3
- removed net Q1.GATE63: C190.1, Q64.1, R127.1, R128.2, ZD64.3
- removed net Q1.GATE64: C193.1, Q65.1, R129.1, R130.2, ZD65.3
- removed net Q1.GATE65: C196.1, Q66.1, R131.1, R132.2, ZD66.3
- removed net Q1.GATE66: C199.1, Q67.1, R133.1, R134.2, ZD67.3
- removed net Q1.GATE67: C202.1, Q68.1, R135.1, R136.2, ZD68.3
- removed net Q1.GATE68: C205.1, Q69.1, R137.1, R138.2, ZD69.3
- removed net Q1.GATE69: C208.1, Q70.1, R139.1, R140.2, ZD70.3
- removed net Q1.GATE70: C211.1, Q71.1, R141.1, R142.2, ZD71.3
- removed net Q1.GATE71: C214.1, Q72.1, R143.1, R144.2, ZD72.3
- removed net VM10: 3.OUT10.1, Q11.2
- removed net VM11: 3.OUT11.1, Q12.2
- removed net VM16: 3.OUT16.1, Q17.2
- removed net VM17: 3.OUT17.1, Q18.2
- removed net VM22: 3.OUT22.1, Q23.2
- removed net VM23: 3.OUT23.1, Q24.2
- removed net VM24: 3.OUT24.1, Q25.2
- removed net VM25: 3.OUT25.1, Q26.2
- removed net VM26: 3.OUT26.1, Q27.2
- removed net VM27: 3.OUT27.1, Q28.2
- removed net VM28: 3.OUT28.1, Q29.2
- removed net VM29: 3.OUT29.1, Q30.2
- removed net VM30: 3.OUT30.1, Q31.2
- removed net VM31: 3.OUT31.1, Q32.2
- removed net VM32: 3.OUT32.1, Q33.2
- removed net VM33: 3.OUT33.1, Q34.2
- removed net VM34: 3.OUT34.1, Q35.2
- removed net VM35: 3.OUT35.1, Q36.2
- removed net VM36: 3.OUT36.1, Q37.2
- removed net VM37: 3.OUT37.1, Q38.2
- removed net VM38: 3.OUT38.1, Q39.2
- removed net VM39: 3.OUT39.1, Q40.2
- removed net VM4: 3.OUT4.1, Q5.2
- removed net VM40: 3.OUT40.1, Q41.2
- removed net VM41: 3.OUT41.1, Q42.2
- removed net VM5: 3.OUT5.1, Q6.2
- removed net VM54: 3.OUT54.1, Q55.2
- removed net VM55: 3.OUT55.1, Q56.2
- removed net VM56: 3.OUT56.1, Q57.2
- removed net VM57: 3.OUT57.1, Q58.2
- removed net VM58: 3.OUT58.1, Q59.2
- removed net VM59: 3.OUT59.1, Q60.2
- removed net VM60: 3.OUT60.1, Q61.2
- removed net VM61: 3.OUT61.1, Q62.2
- removed net VM62: 3.OUT62.1, Q63.2
- removed net VM63: 3.OUT63.1, Q64.2
- removed net VM64: 3.OUT64.1, Q65.2
- removed net VM65: 3.OUT65.1, Q66.2
- removed net VM66: 3.OUT66.1, Q67.2
- removed net VM67: 3.OUT67.1, Q68.2
- removed net VM68: 3.OUT68.1, Q69.2
- removed net VM69: 3.OUT69.1, Q70.2
- removed net VM70: 3.OUT70.1, Q71.2
- removed net VM71: 3.OUT71.1, Q72.2
Routing:
- net GND70: track 17.6 -> 0.00 mm
- net GND64: track 17.6 -> 0.00 mm
- net GND40: track 17.6 -> 0.00 mm
- net GND69: track 17.6 -> 0.00 mm
- net GND68: track 17.6 -> 0.00 mm
- net GND63: track 17.6 -> 0.00 mm
- net GND62: track 17.6 -> 0.00 mm
- net GND39: track 17.6 -> 0.00 mm
- net GND38: track 17.6 -> 0.00 mm
- net GND71: track 17.6 -> 0.00 mm
- net GND67: track 17.6 -> 0.00 mm
- net GND66: track 17.6 -> 0.00 mm
- net GND65: track 17.6 -> 0.00 mm
- net GND61: track 17.6 -> 0.00 mm
- net GND60: track 17.6 -> 0.00 mm
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Other:
- board size 100 x 90 mm -> 40 x 60 mm
