File: 202103 - PCB Fuse Traces/PCB Fuse Traces.sch (EAGLE design)
At the start: 8 parts

Commit message: 20210315
Parts:
- added F10: (no value), nolan:FUSEDD
- added F11: (no value), nolan:FUSEA0
- added F12: (no value), nolan:FUSEA1
- added F13: (no value), nolan:FUSEA3
- added F14: (no value), nolan:FUSEB1
- added F15: (no value), nolan:FUSEB2
- added F16: (no value), nolan:FUSEB3
- added F17: (no value), nolan:FUSEB4
- added F18: (no value), nolan:FUSE1206
- added F19: (no value), nolan:FUSE0805
- added F20: (no value), nolan:FUSE0603
- added F5: (no value), nolan:FUSEB
- added F6: (no value), nolan:FUSEBB
- added F7: (no value), nolan:FUSEC
- added F8: (no value), nolan:FUSECC
- added F9: (no value), nolan:FUSED
- added FH10, FH11, FH12, FH13, FH14, FH15, FH16, FH17, FH18, FH19, FH20, FH5, FH6, FH7, FH8, FH9: (no value), nolan:FUSE_HOLDER36MM
- F1: device nolan:FUSE0603 -> nolan:FUSEA
- F2: device nolan:FUSE0805 -> nolan:FUSEAA
- F3: device nolan:FUSE1206 -> nolan:FUSEAAA
- F4: device nolan:FUSE3X10 -> nolan:FUSEAAAA
Connections:
- new net N$10: F6.1, FH6A.1
- new net N$11: F7.1, FH7A.1
- new net N$12: F8.1, FH8A.1
- new net N$13: F5.2, FH5B.1
- new net N$14: F6.2, FH6B.1
- new net N$15: F7.2, FH7B.1
- new net N$16: F8.2, FH8B.1
- new net N$17: F9.1, FH9A.1
- new net N$18: F10.1, FH10A.1
- new net N$19: F11.1, FH11A.1
- new net N$20: F12.1, FH12A.1
- new net N$21: F9.2, FH9B.1
- new net N$22: F10.2, FH10B.1
- new net N$23: F11.2, FH11B.1
- new net N$24: F12.2, FH12B.1
- new net N$25: F13.1, FH13A.1
- new net N$26: F14.1, FH14A.1
- new net N$27: F15.1, FH15A.1
- new net N$28: F16.1, FH16A.1
- new net N$29: F13.2, FH13B.1
- new net N$30: F14.2, FH14B.1
- new net N$31: F15.2, FH15B.1
- new net N$32: F16.2, FH16B.1
- new net N$33: F17.1, FH17A.1
- new net N$34: F18.1, FH18A.1
- new net N$35: F19.1, FH19A.1
- new net N$36: F20.1, FH20A.1
- new net N$37: F17.2, FH17B.1
- new net N$38: F18.2, FH18B.1
- new net N$39: F19.2, FH19B.1
- new net N$40: F20.2, FH20B.1
- new net N$9: F5.1, FH5A.1
Other:
- moved on the sheet: F1, F2, F3, F4, FH1A, FH1B, FH2A, FH2B, FH3A, FH3B, FH4A, FH4B
